File: Robert/schematics/_autosave-schematics.kicad_pcb (KiCad board)
At the start: 2 copper layers, 120.7 x 43.2 mm, 31 parts, among them J1 STEPPER_L, J2 STEPPER_R, J3 BMI160 Module, J4 POWER, J5 Conn_02x08_Odd_Even, J6 SDD1306, J7 VREG, SW1 MOTOR_L_0, SW10 SW_Push, SW2 MOTOR_L_1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

Commit message: pcb done, double check needed
Parts:
- renumbered G*** to ?
Routing:
- net GND: track 0.00 -> 30.7 mm
- net Net-(A1-~{ENABLE}): track 125.1 -> 105.1 mm
- net Net-(A1-VMOT): track 96.1 -> 98.5 mm
- net Net-(A1-M1): track 46.8 -> 47.6 mm
- net Net-(A2-STEP): track 68.4 -> 67.6 mm
- net Net-(U1-IO35): track 108.7 -> 109.2 mm
Changed lines of the file:
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@@
     (at 114.554 84.582 180)
     (attr board_only exclude_from_pos_files exclude_from_bom)
-    (fp_text reference "G***" (at 0 0) (layer "B.SilkS")
+    (fp_text reference "" (at 0 0) (layer "B.SilkS")
         (effects (font (size 1.5 1.5) (thickness 0.3)) (justify mirror))
     )
@@
     (effects (font (size 2 2) (thickness 0.15)) (justify left bottom mirror))
   )
-  (segment (start 166.37 74.92) (end 166.37 73.87) (width 0.25) (layer "B.Cu") (net 1))
-  (segment (start 104.617 65.247) (end 104.617 79.827) (width 0.25) (layer "B.Cu") (net 1))
-  (segment (start 166.37 73.87) (end 157.27 64.77) (width 0.25) (layer "B.Cu") (net 1))
-  (segment (start 157.27 64.77) (end 104.14 64.77) (width 0.25) (layer "B.Cu") (net 1))
+  (segment (start 119.857 87.813) (end 119.857 65.955749) (width 0.25) (layer "B.Cu") (net 1))
+  (segment (start 166.37 73.87) (end 166.37 74.92) (width 0.25) (layer "B.Cu") (net 1))
+  (segment (start 116.23 91.44) (end 119.857 87.813) (width 0.25) (layer "B.Cu") (net 1))
+  (segment (start 121.042749 64.77) (end 157.27 64.77) (width 0.25) (layer "B.Cu") (net 1))
   (segment (start 166.37 74.92) (end 167.495 76.045) (width 0.25) (layer "B.Cu") (net 1))
+  (segment (start 157.27 64.77) (end 166.37 73.87) (width 0.25) (layer "B.Cu") (net 1))
   (segment (start 167.495 76.045) (end 190.655 76.045) (width 0.25) (layer "B.Cu") (net 1))
+  (segment (start 119.857 65.955749) (end 121.042749 64.77) (width 0.25) (layer "B.Cu") (net 1))
   (segment (start 190.655 76.045) (end 191.77 74.93) (width 0.25) (layer "B.Cu") (net 1))
-  (segment (start 104.617 79.827) (end 116.23 91.44) (width 0.25) (layer "B.Cu") (net 1))
-  (segment (start 104.14 64.77) (end 104.617 65.247) (width 0.25) (layer "B.Cu") (net 1))
   (segment (start 167.65 82.5075) (end 175.27 82.5075) (width 0.25) (layer "F.Cu") (net 2))
   (segment (start 176.395 81.3825) (end 187.8575 81.3825) (width 0.25) (layer "F.Cu") (net 2))
@@
   (segment (start 175.27 82.5075) (end 176.395 81.3825) (width 0.25) (layer "F.Cu") (net 2))
   (segment (start 187.8575 81.3825) (end 194.31 74.93) (width 0.25) (layer "F.Cu") (net 2))
-  (segment (start 171.45 74.92) (end 174 77.47) (width 0.25) (layer "F.Cu") (net 3))
-  (segment (start 174 77.47) (end 186.98 77.47) (width 0.25) (layer "F.Cu") (net 3))
+  (segment (start 175.016 78.486) (end 185.964 78.486) (width 0.25) (layer "F.Cu") (net 3))
   (segment (start 189.2725 82.5075) (end 196.85 74.93) (width 0.25) (layer "F.Cu") (net 3))
   (segment (start 181.6525 82.5075) (end 189.2725 82.5075) (width 0.25) (layer "F.Cu") (net 3))
-  (segment (start 190.645 73.805) (end 195.725 73.805) (width 0.25) (layer "F.Cu") (net 3))
-  (segment (start 186.98 77.47) (end 190.645 73.805) (width 0.25) (layer "F.Cu") (net 3))
+  (segment (start 171.45 74.92) (end 175.016 78.486) (width 0.25) (layer "F.Cu") (net 3))
+  (segment (start 185.964 78.486) (end 190.645 73.805) (width 0.25) (layer "F.Cu") (net 3))
   (segment (start 195.725 73.805) (end 196.85 74.93) (width 0.25) (layer "F.Cu") (net 3))
+  (segment (start 190.645 73.805) (end 195.725 73.805) (width 0.25) (layer "F.Cu") (net 3))
+  (segment (start 173.99 74.92) (end 173.99 74.93) (width 0.25) (layer "F.Cu") (net 4))
+  (segment (start 172.73 90.1275) (end 173.855 91.2525) (width 0.25) (layer "B.Cu") (net 4))
+  (segment (start 173.855 91.2525) (end 185.6075 91.2525) (width 0.25) (layer "B.Cu") (net 4))
+  (segment (start 166.525 91.2525) (end 162.56 87.2875) (width 0.25) (layer "B.Cu") (net 4))
+  (segment (start 172.73 90.1275) (end 171.605 91.2525) (width 0.25) (layer "B.Cu") (net 4))
+  (segment (start 185.6075 91.2525) (end 186.7325 90.1275) (width 0.25) (layer "B.Cu") (net 4))
+  (segment (start 171.605 91.2525) (end 166.525 91.2525) (width 0.25) (layer "B.Cu") (net 4))
+  (segment (start 173.99 74.92) (end 176.53 74.92) (width 0.25) (layer "B.Cu") (net 4))
+  (segment (start 162.56 87.2875) (end 162.56 86.36) (width 0.25) (layer "B.Cu") (net 4))
   (segment (start 209.55 74.93) (end 198.998299 64.378299) (width 0.25) (layer "F.Cu") (net 5))
   (segment (start 117.891701 64.378299) (end 116.23 66.04) (width 0.25) (layer "F.Cu") (net 5))
@@
   (segment (start 176.53 62.22) (end 176.53 55.562) (width 0.4) (layer "F.Cu") (net 13))
   (segment (start 176.53 55.562) (end 176.72 55.372) (width 0.4) (layer "F.Cu") (net 13))
+  (segment (start 185.918 51.816) (end 183.637 54.097) (width 0.4) (layer "F.Cu") (net 14))
   (segment (start 163.739166 57.19) (end 166.37 59.820834) (width 0.25) (layer "F.Cu") (net 14))
   (segment (start 147.55 57.19) (end 147.32 56.96) (width 0.4) (layer "F.Cu") (net 14))
-  (segment (start 210.75 62.8) (end 210.75 59.62) (width 0.4) (layer "F.Cu") (net 14))
-  (segment (start 184.394 53.34) (end 183.637 54.097) (width 0.4) (layer "F.Cu") (net 14))
+  (segment (start 217.17 69.22) (end 210.75 62.8) (width 0.4) (layer "F.Cu") (net 14))
   (segment (start 161.29 57.19) (end 163.739166 57.19) (width 0.25) (layer "F.Cu") (net 14))
   (segment (start 153.67 57.19) (end 161.29 57.19) (width 0.4) (layer "F.Cu") (net 14))
   (segment (start 172.093834 54.097) (end 166.37 59.820834) (width 0.4) (layer "F.Cu") (net 14))
-  (segment (start 210.75 59.62) (end 204.47 53.34) (width 0.4) (layer "F.Cu") (net 14))
   (segment (start 166.37 59.820834) (end 166.37 62.22) (width 0.4) (layer "F.Cu") (net 14))
   (segment (start 183.637 54.097) (end 172.093834 54.097) (width 0.4) (layer "F.Cu") (net 14))
   (segment (start 153.67 57.19) (end 147.55 57.19) (width 0.4) (layer "F.Cu") (net 14))
+  (segment (start 210.75 57.588) (end 204.978 51.816) (width 0.4) (layer "F.Cu") (net 14))
   (segment (start 191.77 62.23) (end 183.637 54.097) (width 0.4) (layer "F.Cu") (net 14))
-  (segment (start 204.47 53.34) (end 184.394 53.34) (width 0.4) (layer "F.Cu") (net 14))
-  (segment (start 217.17 69.22) (end 210.75 62.8) (width 0.4) (layer "F.Cu") (net 14))
+  (segment (start 204.978 51.816) (end 185.918 51.816) (width 0.4) (layer "F.Cu") (net 14))
+  (segment (start 210.75 62.8) (end 210.75 57.588) (width 0.4) (layer "F.Cu") (net 14))
   (segment (start 179.07 62.22) (end 179.07 55.722) (width 0.4) (layer "F.Cu") (net 15))
   (segment (start 179.07 55.722) (end 178.72 55.372) (width 0.4) (layer "F.Cu") (net 15))
@@
   (segment (start 213.65 83.11) (end 213.65 89.61) (width 0.25) (layer "F.Cu") (net 26))
   (segment (start 160.02 69.85) (end 158.895 70.975) (width 0.25) (layer "B.Cu") (net 26))
-  (segment (start 133.865 70.975) (end 128.93 66.04) (width 0.25) (layer "B.Cu") (net 26))
   (segment (start 201.028833 91.295) (end 198.488833 88.755) (width 0.25) (layer "B.Cu") (net 26))
-  (segment (start 211.965 91.295) (end 201.028833 91.295) (width 0.25) (layer "B.Cu") (net 26))
-  (segment (start 198.488833 88.755) (end 168.765 88.755) (width 0.25) (layer "B.Cu") (net 26))
-  (segment (start 158.895 70.975) (end 158.75 70.975) (width 0.25) (layer "B.Cu") (net 26))
-  (segment (start 168.765 88.755) (end 158.75 78.74) (width 0.25) (layer "B.Cu") (net 26))
-  (segment (start 158.75 78.74) (end 158.75 70.975) (width 0.25) (layer "B.Cu") (net 26))
+  (segment (start 133.865 70.975) (end 128.93 66.04) (width 0.25) (layer "B.Cu") (net 26))
   (segment (start 213.65 89.61) (end 211.965 91.295) (width 0.25) (layer "B.Cu") (net 26))
-  (segment (start 158.75 70.975) (end 133.865 70.975) (width 0.25) (layer "B.Cu") (net 26))
+  (segment (start 158.895 70.975) (end 158.75 70.975) (width 0.25) (layer "B.Cu") (net 26))
+  (segment (start 157.48 77.47) (end 168.765 88.755) (width 0.25) (layer "B.Cu") (net 26))
+  (segment (start 158.75 70.975) (end 157.48 70.975) (width 0.25) (layer "B.Cu") (net 26))
+  (segment (start 157.48 70.975) (end 133.865 70.975) (width 0.25) (layer "B.Cu") (net 26))
+  (segment (start 198.488833 88.755) (end 168.765 88.755) (width 0.25) (layer "B.Cu") (net 26))
+  (segment (start 211.965 91.295) (end 201.028833 91.295) (width 0.25) (layer "B.Cu") (net 26))
+  (segment (start 157.48 70.975) (end 157.48 77.47) (width 0.25) (layer "B.Cu") (net 26))
   (segment (start 203.49 83.11) (end 203.49 89.61) (width 0.25) (layer "F.Cu") (net 27))
   (segment (start 157.48 68.58) (end 156.21 69.85) (width 0.25) (layer "B.Cu") (net 27))
@@
   (segment (start 156.21 69.85) (end 135.28 69.85) (width 0.25) (layer "B.Cu") (net 27))
   (segment (start 161.29 79.060991) (end 161.29 69.529009) (width 0.25) (layer "B.Cu") (net 27))
-  (segment (start 175.405 73.805) (end 168.91 67.31) (width 0.25) (layer "F.Cu") (net 33))
   (segment (start 120.04 67.31) (end 118.77 66.04) (width 0.25) (layer "F.Cu") (net 33))
-  (segment (start 175.405 75.385991) (end 175.405 73.805) (width 0.25) (layer "F.Cu") (net 33))
-  (segment (start 168.91 67.31) (end 120.04 67.31) (width 0.25) (layer "F.Cu") (net 33))
-  (segment (start 180.485 76.045) (end 176.064009 76.045) (width 0.25) (layer "F.Cu") (net 33))
-  (segment (start 176.064009 76.045) (end 175.405 75.385991) (width 0.25) (layer "F.Cu") (net 33))
-  (segment (start 181.61 74.92) (end 180.485 76.045) (width 0.25) (layer "F.Cu") (net 33))
+  (segment (start 175.903604 67.31) (end 120.04 67.31) (width 0.25) (layer "F.Cu") (net 33))
+  (segment (start 181.61 74.92) (end 181.61 73.016396) (width 0.25) (layer "F.Cu") (net 33))
+  (segment (start 181.61 73.016396) (end 175.903604 67.31) (width 0.25) (layer "F.Cu") (net 33))
   (segment (start 148.685 73.755) (end 149.285 74.355) (width 0.25) (layer "F.Cu") (net 36))
   (segment (start 149.285 74.355) (end 151.788148 74.355) (width 0.25) (layer "F.Cu") (net 36))
