File: Robert/schematics/schematics.kicad_pcb (KiCad board)
At the start: 2 copper layers, 120.7 x 43.2 mm, 31 parts, among them J1 STEPPER_L, J2 STEPPER_R, J3 BMI160 Module, J4 POWER, J5 Conn_02x08_Odd_Even, J6 SDD1306, J7 VREG, SW1 MOTOR_L_0, SW10 SW_Push, SW2 MOTOR_L_1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

Commit message: revised pcb
Parts:
- moved J6 7.62 mm to (105.4, 62.2), turned to 180 degrees
Connections:
- A1 pad 10: Net-(A1-~{FAULT}) -> unconnected-(A1-~{FAULT}-Pad10)
- A1 pad 6: Net-(A1-~{FAULT}) -> Net-(A1-~{SLEEP})
- A2 pad 10: Net-(A2-~{FAULT}) -> unconnected-(A2-~{FAULT}-Pad10)
- A2 pad 6: Net-(A2-~{FAULT}) -> Net-(A1-~{SLEEP})
- J3 pad 2: Net-(J3-Pin_2) -> Net-(A1-~{SLEEP})
- J5 pad 3: Net-(J3-Pin_2) -> Net-(A1-~{SLEEP})
- J5 pad 4: Net-(J3-Pin_2) -> Net-(A1-~{SLEEP})
- J6 pad 2: Net-(J3-Pin_2) -> Net-(A1-~{SLEEP})
- J7 pad 2: Net-(J3-Pin_2) -> Net-(A1-~{SLEEP})
- R2 pad 1: Net-(J3-Pin_2) -> Net-(A1-~{SLEEP})
- R4 pad 1: Net-(J3-Pin_2) -> Net-(A1-~{SLEEP})
- SW1 pad 4: Net-(J3-Pin_2) -> Net-(A1-~{SLEEP})
- SW10 pad 2: Net-(J3-Pin_2) -> Net-(A1-~{SLEEP})
- SW2 pad 4: Net-(J3-Pin_2) -> Net-(A1-~{SLEEP})
- SW9 pad 2: Net-(J3-Pin_2) -> Net-(A1-~{SLEEP})
- U1 pad 16: Net-(J3-Pin_2) -> Net-(A1-~{SLEEP})
Routing:
- net Net-(A1-~{SLEEP}): track 0.00 -> 293.6 mm
- net Net-(J3-Pin_2): track 258.7 -> 0.00 mm
- net Net-(A2-~{FAULT}): track 13.8 -> 0.00 mm
- net Net-(A1-~{FAULT}): track 13.8 -> 0.00 mm
- net Net-(A1-~{ENABLE}): track 125.1 -> 116.7 mm
- net Net-(J3-Pin_3): track 81.3 -> 83.8 mm
- net Net-(A2-STEP): track 68.4 -> 66.5 mm
- net Net-(J3-Pin_4): track 90.3 -> 89.0 mm
- net Net-(A1-M1): track 46.8 -> 47.8 mm
