File: Robert/schematics/schematics.kicad_sch (KiCad schematic)
At the start: 28 parts, among them J1 STEPPER_L, J2 STEPPER_R, J3 BMI160 Module, J4 POWER, J5 SD, J6 SDD1306, J7 VREG, SW1 MOTOR_L_0, SW10 SW_Push, SW2 MOTOR_L_1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

Commit message: pcb done, double check needed
Parts:
- removed J5: SD, Connector_PinHeader_2.54mm:PinHeader_2x08_P2.54mm_Vertical, symbol Connector_Generic:Conn_02x08_Counter_Clockwise
- removed R5, R6, R7, R8: 330k, Resistor_THT:R_Axial_DIN0207_L6.3mm_D2.5mm_P2.54mm_Vertical, symbol Device:R
- removed SW7: MOTOR_R_0, Button_Switch_THT:SW_DIP_SPSTx04_Slide_9.78x12.34mm_W7.62mm_P2.54mm, symbol Switch:SW_DIP_x04
- removed SW8: MOTOR_R_1, Button_Switch_THT:SW_DIP_SPSTx04_Slide_9.78x12.34mm_W7.62mm_P2.54mm, symbol Switch:SW_DIP_x04
- added J5: Conn_02x08_Odd_Even, Connector_PinHeader_2.54mm:PinHeader_2x08_P2.54mm_Vertical, symbol Connector_Generic:Conn_02x08_Odd_Even
- added SW3: SW_SPDT, boards:SW_Toggle_Blue_wSlots, symbol Switch:SW_SPDT
Connections:
- net GND: now also A1.15 (GND), A2.15 (GND), J5.1 (Pin_1), J5.16 (Pin_16), J5.2 (Pin_2); no longer A1.7 (STEP), A2.7 (STEP), R2.1, R4.1
- net at A2.10 (~{FAULT}): now also A2.6 (~{SLEEP}); no longer J1.1 (Pin_1)
- net at A2.11 (A1): now also J1.4 (Pin_4); no longer J1.2 (Pin_2)
- net at A2.13 (B2): now also J1.2 (Pin_2); no longer J1.4 (Pin_4)
- net at A2.2 (M0), SW1.5, SW1.6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: now also A1.2 (M0)
- net at A2.3 (M1), SW2.5, SW2.6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: now also A1.3 (M1)
- net at C1.1, C2.1, J7.1 (Pin_1): now also A1.16 (VMOT), A2.16 (VMOT), SW3.2 (B); no longer A1.9 (VMOT), A2.9 (VMOT), J4.1 (Pin_1)
- net at J3.2 (Pin_2), J6.2 (Pin_2), J7.2 (Pin_2)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: now also R2.1, R4.1, J5.3 (Pin_3), J5.4 (Pin_4)
- net at U1.25 (IO19): now also J5.13 (Pin_13), J5.14 (Pin_14)
- net at U1.24 (IO18): now also J5.11 (Pin_11), J5.12 (Pin_12)
- net at U1.30 (IO23): now also J5.10 (Pin_10), J5.9 (Pin_9)
- net at U1.23 (IO5): now also J5.7 (Pin_7), J5.8 (Pin_8)
- net at A1.10 (~{FAULT}): now also A1.6 (~{SLEEP}); no longer J2.1 (Pin_1)
- net at A1.11 (A1): now also J2.4 (Pin_4); no longer J2.2 (Pin_2)
- net at A1.13 (B2): now also J2.2 (Pin_2); no longer J2.4 (Pin_4)
- new net: A2.14 (B1), J1.1 (Pin_1)
- new net: A1.14 (B1), J2.1 (Pin_1)
- new net: J4.1 (Pin_1), SW3.3 (C)
- no-connect marks 21 -> 15
Other:
- moved on the sheet: J1, J2, J4, R1, R2, R3, R4, SW1, SW2

Commit message: revised pcb
Connections:
- net at J3.2 (Pin_2), J5.3 (Pin_3), J5.4 (Pin_4)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: now also A1.6 (~{SLEEP}), A2.6 (~{SLEEP})
- net at A2.10 (~{FAULT}): no longer A2.6 (~{SLEEP})
- net at A1.10 (~{FAULT}): no longer A1.6 (~{SLEEP})
- no-connect marks 15 -> 17
Changed lines of the file:
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@@
   (junction (at 168.91 132.08) (diameter 0) (color 0 0 0 0)
   )
+  (junction (at 190.5 68.58) (diameter 0) (color 0 0 0 0)
+  )
   (junction (at 158.75 147.32) (diameter 0) (color 0 0 0 0)
   )
@@
   )
   (junction (at 132.08 201.93) (diameter 0) (color 0 0 0 0)
+  )
+  (junction (at 208.28 118.11) (diameter 0) (color 0 0 0 0)
   )
   (junction (at 193.04 134.62) (diameter 0) (color 0 0 0 0)
@@
   (no_connect (at 54.61 107.95))
   (no_connect (at 72.39 118.11))
+  (no_connect (at 210.82 115.57))
   (no_connect (at 72.39 128.27))
   (no_connect (at 41.91 113.03))
@@
   (no_connect (at 153.67 43.18))
   (no_connect (at 72.39 166.37))
+  (no_connect (at 210.82 170.18))
   (no_connect (at 72.39 163.83))
-  (wire (pts (xy 209.55 170.18) (xy 209.55 172.72))
-    (stroke (width 0) (type default))
-  )
   (wire (pts (xy 233.68 180.34) (xy 236.22 180.34))
     (stroke (width 0) (type default))
@@
     (stroke (width 0) (type default))
   )
-  (wire (pts (xy 209.55 115.57) (xy 210.82 115.57))
-    (stroke (width 0) (type default))
-  )
   (wire (pts (xy 166.37 132.08) (xy 168.91 132.08))
     (stroke (width 0) (type default))
@@
     (stroke (width 0) (type default))
   )
+  (wire (pts (xy 210.82 172.72) (xy 208.28 172.72))
+    (stroke (width 0) (type default))
+  )
   (wire (pts (xy 99.06 215.9) (xy 99.06 213.36))
     (stroke (width 0) (type default))
@@
     (stroke (width 0) (type default))
   )
+  (wire (pts (xy 190.5 68.58) (xy 208.28 68.58))
+    (stroke (width 0) (type default))
+  )
   (wire (pts (xy 137.16 81.28) (xy 163.83 81.28))
     (stroke (width 0) (type default))
@@
     (stroke (width 0) (type default))
   )
-  (wire (pts (xy 209.55 115.57) (xy 209.55 118.11))
-    (stroke (width 0) (type default))
-  )
   (wire (pts (xy 77.47 201.93) (xy 80.01 201.93))
     (stroke (width 0) (type default))
@@
     (stroke (width 0) (type default))
   )
+  (wire (pts (xy 208.28 118.11) (xy 210.82 118.11))
+    (stroke (width 0) (type default))
+  )
   (wire (pts (xy 149.86 125.73) (xy 210.82 125.73))
     (stroke (width 0) (type default))
@@
     (stroke (width 0) (type default))
   )
-  (wire (pts (xy 209.55 118.11) (xy 210.82 118.11))
-    (stroke (width 0) (type default))
-  )
   (wire (pts (xy 171.45 77.47) (xy 171.45 82.55))
     (stroke (width 0) (type default))
@@
     (stroke (width 0) (type default))
   )
+  (wire (pts (xy 208.28 68.58) (xy 208.28 118.11))
+    (stroke (width 0) (type default))
+  )
   (wire (pts (xy 201.93 191.77) (xy 201.93 201.93))
     (stroke (width 0) (type default))
@@
     (stroke (width 0) (type default))
   )
-  (wire (pts (xy 210.82 172.72) (xy 209.55 172.72))
-    (stroke (width 0) (type default))
-  )
   (wire (pts (xy 91.44 93.98) (xy 105.41 93.98))
     (stroke (width 0) (type default))
@@
     (stroke (width 0) (type default))
   )
-  (wire (pts (xy 210.82 170.18) (xy 209.55 170.18))
-    (stroke (width 0) (type default))
-  )
   (wire (pts (xy 185.42 189.23) (xy 187.96 189.23))
     (stroke (width 0) (type default))
@@
     (stroke (width 0) (type default))
   )
+  (wire (pts (xy 208.28 172.72) (xy 208.28 118.11))
+    (stroke (width 0) (type default))
+  )
